Commit message: Cleanup of gazebo test code which didn't work

File: subwoofer_model/urdf/imports/builders.xacro (robot description, xacro)
@@ -188,58 +188,4 @@
             rpy="0 0 0"
             xyz="${0*scale} ${-79*scale} ${0*scale}" />
-        <!-- Camera -->
-        <link name="camera_link">
-            <inertial>
-                <mass value="0.010"/>
-                <inertia ixx="1e-6" ixy="0.0" ixz="0.0" iyy="1e-6" iyz="0.0" izz="1e-6"/>
-            </inertial>
-            <visual>
-                <origin rpy="0 0 0" xyz="0 0 0"/>
-                <geometry>
-                    <box size="0.01 0.03 0.03"/>
-                </geometry>
-                <material name="RED"/>
-            </visual>
-            <collision>
-                <origin rpy="0 0 0" xyz="0 0 0"/>
-                <geometry>
-                    <box size="0.01 0.03 0.03"/>
-                </geometry>
-            </collision>
-        </link>
-        <xacro:create_fixed_joint
-            parent="nose_chassis"
-            child="camera_link"
-            rpy="0 0 0"
-            xyz="${0*scale} ${0*scale} ${0*scale}" />
-        <link name="camera_optical_link"></link>
-        <xacro:create_fixed_joint
-            parent="camera_link"
-            child="camera_optical_link"
-            rpy="-1.57075 0 -1.57075"
-            xyz="${0*scale} ${0*scale} ${0*scale}" />
-        <gazebo reference="camera_link">
-            <material>Gazebo/Red</material>
-            <sensor type="camera" name="camera">
-                <pose> 0 0 0 0 0 0 </pose>
-                <visualize>true</visualize>
-                <update_rate>10</update_rate>
-                <camera>
-                    <horizontal_fov>1.089</horizontal_fov>
-                    <image>
-                        <format>R8G8B8</format>
-                        <width>640</width>
-                        <height>480</height>
-                    </image>
-                    <clip>
-                        <near>0.05</near>
-                        <far>8.0</far>
-                    </clip>
-                </camera>
-                <plugin name="camera_controller" filename="libgazebo_ros_camera.so">
-                    <frame_name>camera_link_optical</frame_name>
-                </plugin>
-            </sensor>
-        </gazebo>
     </xacro:macro>
     <!-- Leg builder -->

File: subwoofer_model/urdf/subwoofer.urdf.xacro (robot description, xacro)
@@ -21,19 +21,3 @@
         name="back_right"
         xyz="${37*scale} ${0*scale} ${7*scale}" />
-  <!-- Joint publish test -->
-  <plugin
-    filename="ignition-gazebo-joint-state-publisher-system"
-    name="ignition::gazebo::systems::JointStatePublisher">
-  </plugin>
-  <plugin
-    filename="ignition-gazebo-joint-controller-system"
-    name="ignition::gazebo::systems::JointController">
-    <joint_name>front_right_hip_servo_to_front_outer_shoulder</joint_name>
-  </plugin>
-  <plugin
-    filename="ignition-gazebo-pose-publisher-system"
-    name="ignition::gazebo::systems::PosePublisher">
-    <publish_link_pose>true</publish_link_pose>
-    <use_pose_vector_msg>true</use_pose_vector_msg>
-  </plugin>
 </robot>
